Commit message: add com

File: ycb_assets/002_master_chef_can/google_16k/002_master_chef_can.urdf (robot description, URDF)
Before this commit: robot 002_master_chef_can, 1 links, 0 joints
Links:
- removed link 002_master_chef_can
- added link base_link, mass 0.1; collision mesh filename=textured_vhacd.obj; visual mesh filename=textured.obj
- added link center_of_mass
Joints:
- added joint base_to_com: type fixed, parent base_link, child center_of_mass, origin xyz=0 0 0.069796 rpy=0 0 0

File: ycb_assets/003_cracker_box/google_16k/003_cracker_box.urdf (robot description, URDF)
Before this commit: robot 003_cracker_box, 1 links, 0 joints
Links:
- removed link 003_cracker_box
- added link base_link, mass 0.1; collision mesh filename=textured_vhacd.obj; visual mesh filename=textured.obj
- added link center_of_mass
Joints:
- added joint base_to_com: type fixed, parent base_link, child center_of_mass, origin xyz=0 0 0.107097 rpy=0 0 0

File: ycb_assets/004_sugar_box/google_16k/004_sugar_box.urdf (robot description, URDF)
Before this commit: robot 004_sugar_box, 1 links, 0 joints
Links:
- removed link 004_sugar_box
- added link base_link, mass 0.1; collision mesh filename=textured_vhacd.obj; visual mesh filename=textured.obj
- added link center_of_mass
Joints:
- added joint base_to_com: type fixed, parent base_link, child center_of_mass, origin xyz=0 0 0.087626 rpy=0 0 0

File: ycb_assets/005_tomato_soup_can/google_16k/005_tomato_soup_can.urdf (robot description, URDF)
Before this commit: robot 005_tomato_soup_can, 1 links, 0 joints
Links:
- removed link 005_tomato_soup_can
- added link base_link, mass 0.1; collision mesh filename=textured_vhacd.obj; visual mesh filename=textured.obj
- added link center_of_mass
Joints:
- added joint base_to_com: type fixed, parent base_link, child center_of_mass, origin xyz=0 0 0.061134 rpy=0 0 0

File: ycb_assets/006_mustard_bottle/google_16k/006_mustard_bottle.urdf (robot description, URDF)
Before this commit: robot 006_mustard_bottle, 1 links, 0 joints
Links:
- removed link 006_mustard_bottle
- added link base_link, mass 0.1; collision mesh filename=textured_vhacd.obj; visual mesh filename=textured.obj
- added link center_of_mass
Joints:
- added joint base_to_com: type fixed, parent base_link, child center_of_mass, origin xyz=0 0 0.080734 rpy=0 0 0

File: ycb_assets/007_tuna_fish_can/google_16k/007_tuna_fish_can.urdf (robot description, URDF)
Before this commit: robot 007_tuna_fish_can, 1 links, 0 joints
Links:
- removed link 007_tuna_fish_can
- added link base_link, mass 0.1; collision mesh filename=textured_vhacd.obj; visual mesh filename=textured.obj
- added link center_of_mass
Joints:
- added joint base_to_com: type fixed, parent base_link, child center_of_mass, origin xyz=0 0 0.014302 rpy=0 0 0

File: ycb_assets/008_pudding_box/google_16k/008_pudding_box.urdf (robot description, URDF)
Before this commit: robot 008_pudding_box, 1 links, 0 joints
Links:
- removed link 008_pudding_box
- added link base_link, mass 0.1; collision mesh filename=textured_vhacd.obj; visual mesh filename=textured.obj
- added link center_of_mass
Joints:
- added joint base_to_com: type fixed, parent base_link, child center_of_mass, origin xyz=0 0 0.018664 rpy=0 0 0

File: ycb_assets/009_gelatin_box/google_16k/009_gelatin_box.urdf (robot description, URDF)
Before this commit: robot 009_gelatin_box, 1 links, 0 joints
Links:
- removed link 009_gelatin_box
- added link base_link, mass 0.1; collision mesh filename=textured_vhacd.obj; visual mesh filename=textured.obj
- added link center_of_mass
Joints:
- added joint base_to_com: type fixed, parent base_link, child center_of_mass, origin xyz=0 0 0.013958 rpy=0 0 0

File: ycb_assets/010_potted_meat_can/google_16k/010_potted_meat_can.urdf (robot description, URDF)
Before this commit: robot 010_potted_meat_can, 1 links, 0 joints
Links:
- removed link 010_potted_meat_can
- added link base_link, mass 0.1; collision mesh filename=textured_vhacd.obj; visual mesh filename=textured.obj
- added link center_of_mass
Joints:
- added joint base_to_com: type fixed, parent base_link, child center_of_mass, origin xyz=0 0 0.050106 rpy=0 0 0

File: ycb_assets/011_banana/google_16k/011_banana.urdf (robot description, URDF)
Before this commit: robot 011_banana, 1 links, 0 joints
Links:
- removed link 011_banana
- added link base_link, mass 0.1; collision mesh filename=textured_vhacd.obj; visual mesh filename=textured.obj
- added link center_of_mass
Joints:
- added joint base_to_com: type fixed, parent base_link, child center_of_mass, origin xyz=0 0 0.016670 rpy=0 0 0

File: ycb_assets/012_strawberry/google_16k/012_strawberry.urdf (robot description, URDF)
Before this commit: robot 012_strawberry, 1 links, 0 joints
Links:
- removed link 012_strawberry
- added link base_link, mass 0.1; collision mesh filename=textured_vhacd.obj; visual mesh filename=textured.obj
- added link center_of_mass
Joints:
- added joint base_to_com: type fixed, parent base_link, child center_of_mass, origin xyz=0 0 0.021076 rpy=0 0 0

File: ycb_assets/013_apple/google_16k/013_apple.urdf (robot description, URDF)
Before this commit: robot 013_apple, 1 links, 0 joints
Links:
- removed link 013_apple
- added link base_link, mass 0.1; collision mesh filename=textured_vhacd.obj; visual mesh filename=textured.obj
- added link center_of_mass
Joints:
- added joint base_to_com: type fixed, parent base_link, child center_of_mass, origin xyz=0 0 0.036490 rpy=0 0 0

File: ycb_assets/014_lemon/google_16k/014_lemon.urdf (robot description, URDF)
Before this commit: robot 014_lemon, 1 links, 0 joints
Links:
- removed link 014_lemon
- added link base_link, mass 0.1; collision mesh filename=textured_vhacd.obj; visual mesh filename=textured.obj
- added link center_of_mass
Joints:
- added joint base_to_com: type fixed, parent base_link, child center_of_mass, origin xyz=0 0 0.026204 rpy=0 0 0

File: ycb_assets/015_peach/google_16k/015_peach.urdf (robot description, URDF)
Before this commit: robot 015_peach, 1 links, 0 joints
Links:
- removed link 015_peach
- added link base_link, mass 0.1; collision mesh filename=textured_vhacd.obj; visual mesh filename=textured.obj
- added link center_of_mass
Joints:
- added joint base_to_com: type fixed, parent base_link, child center_of_mass, origin xyz=0 0 0.028322 rpy=0 0 0

File: ycb_assets/016_pear/google_16k/016_pear.urdf (robot description, URDF)
Before this commit: robot 016_pear, 1 links, 0 joints
Links:
- removed link 016_pear
- added link base_link, mass 0.1; collision mesh filename=textured_vhacd.obj; visual mesh filename=textured.obj
- added link center_of_mass
Joints:
- added joint base_to_com: type fixed, parent base_link, child center_of_mass, origin xyz=0 0 0.028412 rpy=0 0 0

File: ycb_assets/017_orange/google_16k/017_orange.urdf (robot description, URDF)
Before this commit: robot 017_orange, 1 links, 0 joints
Links:
- removed link 017_orange
- added link base_link, mass 0.1; collision mesh filename=textured_vhacd.obj; visual mesh filename=textured.obj
- added link center_of_mass
Joints:
- added joint base_to_com: type fixed, parent base_link, child center_of_mass, origin xyz=0 0 0.033553 rpy=0 0 0

File: ycb_assets/018_plum/google_16k/018_plum.urdf (robot description, URDF)
Before this commit: robot 018_plum, 1 links, 0 joints
Links:
- removed link 018_plum
- added link base_link, mass 0.1; collision mesh filename=textured_vhacd.obj; visual mesh filename=textured.obj
- added link center_of_mass
Joints:
- added joint base_to_com: type fixed, parent base_link, child center_of_mass, origin xyz=0 0 0.023377 rpy=0 0 0

File: ycb_assets/019_pitcher_base/google_16k/019_pitcher_base.urdf (robot description, URDF)
Before this commit: robot 019_pitcher_base, 1 links, 0 joints
Links:
- removed link 019_pitcher_base
- added link base_link, mass 0.1; collision mesh filename=textured_vhacd.obj; visual mesh filename=textured.obj
- added link center_of_mass
Joints:
- added joint base_to_com: type fixed, parent base_link, child center_of_mass, origin xyz=0 0 0.141793 rpy=0 0 0

File: ycb_assets/021_bleach_cleanser/google_16k/021_bleach_cleanser.urdf (robot description, URDF)
Before this commit: robot 021_bleach_cleanser, 1 links, 0 joints
Links:
- removed link 021_bleach_cleanser
- added link base_link, mass 0.1; collision mesh filename=textured_vhacd.obj; visual mesh filename=textured.obj
- added link center_of_mass
Joints:
- added joint base_to_com: type fixed, parent base_link, child center_of_mass, origin xyz=0 0 0.113166 rpy=0 0 0

File: ycb_assets/022_windex_bottle/google_16k/022_windex_bottle.urdf (robot description, URDF)
Before this commit: robot 022_windex_bottle, 1 links, 0 joints
Links:
- removed link 022_windex_bottle
- added link base_link, mass 0.1; collision mesh filename=textured_vhacd.obj; visual mesh filename=textured.obj
- added link center_of_mass
Joints:
- added joint base_to_com: type fixed, parent base_link, child center_of_mass, origin xyz=0 0 0.111863 rpy=0 0 0
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
Commit message: obb

File: ycb_assets/002_master_chef_can/google_16k/002_master_chef_can.urdf (robot description, URDF)
Before this commit: robot 002_master_chef_can, 2 links, 1 joints
Links:
- added link obb_center
Joints:
- added joint base_to_obb: type fixed, parent base_link, child obb_center, origin xyz=-0.000196 -0.000103 0.069898 rpy=0 0 0
- joint base_to_com: origin xyz=0 0 0.069796 rpy=0 0 0 -> xyz=0.000000 0.000000 0.069796 rpy=0 0 0

File: ycb_assets/003_cracker_box/google_16k/003_cracker_box.urdf (robot description, URDF)
Before this commit: robot 003_cracker_box, 2 links, 1 joints
Links:
- added link obb_center
Joints:
- added joint base_to_obb: type fixed, parent base_link, child obb_center, origin xyz=0.002146 -0.000256 0.103476 rpy=0 0 0
- joint base_to_com: origin xyz=0 0 0.107097 rpy=0 0 0 -> xyz=0.000000 0.000000 0.107097 rpy=0 0 0

File: ycb_assets/004_sugar_box/google_16k/004_sugar_box.urdf (robot description, URDF)
Before this commit: robot 004_sugar_box, 2 links, 1 joints
Links:
- added link obb_center
Joints:
- added joint base_to_obb: type fixed, parent base_link, child obb_center, origin xyz=0.001035 -0.000133 0.087886 rpy=0 0 0
- joint base_to_com: origin xyz=0 0 0.087626 rpy=0 0 0 -> xyz=0.000000 0.000000 0.087626 rpy=0 0 0

File: ycb_assets/005_tomato_soup_can/google_16k/005_tomato_soup_can.urdf (robot description, URDF)
Before this commit: robot 005_tomato_soup_can, 2 links, 1 joints
Links:
- added link obb_center
Joints:
- added joint base_to_obb: type fixed, parent base_link, child obb_center, origin xyz=0.000007 -0.000268 0.051006 rpy=0 0 0
- joint base_to_com: origin xyz=0 0 0.061134 rpy=0 0 0 -> xyz=0.000000 0.000000 0.061134 rpy=0 0 0

File: ycb_assets/006_mustard_bottle/google_16k/006_mustard_bottle.urdf (robot description, URDF)
Before this commit: robot 006_mustard_bottle, 2 links, 1 joints
Links:
- added link obb_center
Joints:
- added joint base_to_obb: type fixed, parent base_link, child obb_center, origin xyz=0.000191 0.000016 0.092391 rpy=0 0 0
- joint base_to_com: origin xyz=0 0 0.080734 rpy=0 0 0 -> xyz=-0.000000 0.000000 0.080734 rpy=0 0 0

File: ycb_assets/007_tuna_fish_can/google_16k/007_tuna_fish_can.urdf (robot description, URDF)
Before this commit: robot 007_tuna_fish_can, 2 links, 1 joints
Links:
- added link obb_center
Joints:
- added joint base_to_obb: type fixed, parent base_link, child obb_center, origin xyz=0.000789 -0.000175 0.013570 rpy=0 0 0
- joint base_to_com: origin xyz=0 0 0.014302 rpy=0 0 0 -> xyz=0.000000 0.000000 0.014302 rpy=0 0 0

File: ycb_assets/008_pudding_box/google_16k/008_pudding_box.urdf (robot description, URDF)
Before this commit: robot 008_pudding_box, 2 links, 1 joints
Links:
- added link obb_center
Joints:
- added joint base_to_obb: type fixed, parent base_link, child obb_center, origin xyz=0.000473 0.000507 0.018315 rpy=0 0 0
- joint base_to_com: origin xyz=0 0 0.018664 rpy=0 0 0 -> xyz=0.000000 -0.000000 0.018664 rpy=0 0 0

File: ycb_assets/009_gelatin_box/google_16k/009_gelatin_box.urdf (robot description, URDF)
Before this commit: robot 009_gelatin_box, 2 links, 1 joints
Links:
- added link obb_center
Joints:
- added joint base_to_obb: type fixed, parent base_link, child obb_center, origin xyz=-0.000114 -0.000203 0.014422 rpy=0 0 0
- joint base_to_com: origin xyz=0 0 0.013958 rpy=0 0 0 -> xyz=0.000000 0.000000 0.013958 rpy=0 0 0

File: ycb_assets/010_potted_meat_can/google_16k/010_potted_meat_can.urdf (robot description, URDF)
Before this commit: robot 010_potted_meat_can, 2 links, 1 joints
Links:
- added link obb_center
Joints:
- added joint base_to_obb: type fixed, parent base_link, child obb_center, origin xyz=-0.000508 -0.000198 0.038512 rpy=0 0 0
- joint base_to_com: origin xyz=0 0 0.050106 rpy=0 0 0 -> xyz=0.000000 0.000000 0.050106 rpy=0 0 0

File: ycb_assets/011_banana/google_16k/011_banana.urdf (robot description, URDF)
Before this commit: robot 011_banana, 2 links, 1 joints
Links:
- added link obb_center
Joints:
- added joint base_to_obb: type fixed, parent base_link, child obb_center, origin xyz=0.003782 -0.008111 0.017946 rpy=0 0 0
- joint base_to_com: origin xyz=0 0 0.016670 rpy=0 0 0 -> xyz=0.000000 -0.000000 0.016670 rpy=0 0 0

File: ycb_assets/012_strawberry/google_16k/012_strawberry.urdf (robot description, URDF)
Before this commit: robot 012_strawberry, 2 links, 1 joints
Links:
- added link obb_center
Joints:
- added joint base_to_obb: type fixed, parent base_link, child obb_center, origin xyz=0.000577 -0.000792 0.022492 rpy=0 0 0
- joint base_to_com: origin xyz=0 0 0.021076 rpy=0 0 0 -> xyz=-0.000000 0.000000 0.021076 rpy=0 0 0

File: ycb_assets/013_apple/google_16k/013_apple.urdf (robot description, URDF)
Before this commit: robot 013_apple, 2 links, 1 joints
Links:
- added link obb_center
Joints:
- added joint base_to_obb: type fixed, parent base_link, child obb_center, origin xyz=0.000210 -0.000064 0.035734 rpy=0 0 0
- joint base_to_com: origin xyz=0 0 0.036490 rpy=0 0 0 -> xyz=0.000000 0.000000 0.036490 rpy=0 0 0

File: ycb_assets/014_lemon/google_16k/014_lemon.urdf (robot description, URDF)
Before this commit: robot 014_lemon, 2 links, 1 joints
Links:
- added link obb_center
Joints:
- added joint base_to_obb: type fixed, parent base_link, child obb_center, origin xyz=0.000181 -0.000368 0.026632 rpy=0 0 0
- joint base_to_com: origin xyz=0 0 0.026204 rpy=0 0 0 -> xyz=-0.000000 0.000000 0.026204 rpy=0 0 0

File: ycb_assets/015_peach/google_16k/015_peach.urdf (robot description, URDF)
Before this commit: robot 015_peach, 2 links, 1 joints
Links:
- added link obb_center
Joints:
- added joint base_to_obb: type fixed, parent base_link, child obb_center, origin xyz=-0.000431 0.000093 0.026309 rpy=0 0 0
- joint base_to_com: origin xyz=0 0 0.028322 rpy=0 0 0 -> xyz=0.000000 0.000000 0.028322 rpy=0 0 0

File: ycb_assets/016_pear/google_16k/016_pear.urdf (robot description, URDF)
Before this commit: robot 016_pear, 2 links, 1 joints
Links:
- added link obb_center
Joints:
- added joint base_to_obb: type fixed, parent base_link, child obb_center, origin xyz=0.003637 0.000150 0.033377 rpy=0 0 0
- joint base_to_com: origin xyz=0 0 0.028412 rpy=0 0 0 -> xyz=0.000000 -0.000000 0.028412 rpy=0 0 0

File: ycb_assets/017_orange/google_16k/017_orange.urdf (robot description, URDF)
Before this commit: robot 017_orange, 2 links, 1 joints
Links:
- added link obb_center
Joints:
- added joint base_to_obb: type fixed, parent base_link, child obb_center, origin xyz=0.000569 0.000453 0.033266 rpy=0 0 0
- joint base_to_com: origin xyz=0 0 0.033553 rpy=0 0 0 -> xyz=0.000000 0.000000 0.033553 rpy=0 0 0

File: ycb_assets/018_plum/google_16k/018_plum.urdf (robot description, URDF)
Before this commit: robot 018_plum, 2 links, 1 joints
Links:
- added link obb_center
Joints:
- added joint base_to_obb: type fixed, parent base_link, child obb_center, origin xyz=0.000406 0.000257 0.025205 rpy=0 0 0
- joint base_to_com: origin xyz=0 0 0.023377 rpy=0 0 0 -> xyz=-0.000000 -0.000000 0.023377 rpy=0 0 0

File: ycb_assets/019_pitcher_base/google_16k/019_pitcher_base.urdf (robot description, URDF)
Before this commit: robot 019_pitcher_base, 2 links, 1 joints
Links:
- added link obb_center
Joints:
- added joint base_to_obb: type fixed, parent base_link, child obb_center, origin xyz=0.005171 -0.000563 0.118717 rpy=0 0 0
- joint base_to_com: origin xyz=0 0 0.141793 rpy=0 0 0 -> xyz=0.000000 0.000000 0.141793 rpy=0 0 0

File: ycb_assets/021_bleach_cleanser/google_16k/021_bleach_cleanser.urdf (robot description, URDF)
Before this commit: robot 021_bleach_cleanser, 2 links, 1 joints
Links:
- added link obb_center
Joints:
- added joint base_to_obb: type fixed, parent base_link, child obb_center, origin xyz=0.000019 -0.001353 0.124309 rpy=0 0 0
- joint base_to_com: origin xyz=0 0 0.113166 rpy=0 0 0 -> xyz=0.000000 0.000000 0.113166 rpy=0 0 0

File: ycb_assets/022_windex_bottle/google_16k/022_windex_bottle.urdf (robot description, URDF)
Before this commit: robot 022_windex_bottle, 2 links, 1 joints
Links:
- added link obb_center
Joints:
- added joint base_to_obb: type fixed, parent base_link, child obb_center, origin xyz=0.001434 0.002731 0.134579 rpy=0 0 0
- joint base_to_com: origin xyz=0 0 0.111863 rpy=0 0 0 -> xyz=0.000000 -0.000000 0.111863 rpy=0 0 0
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
Commit message: add mass prop

File: ycb_assets/002_master_chef_can/google_16k/002_master_chef_can.urdf (robot description, URDF)
Before this commit: robot 002_master_chef_can, 3 links, 2 joints
Links:
- link base_link: mass 0.1 -> 0.414

File: ycb_assets/003_cracker_box/google_16k/003_cracker_box.urdf (robot description, URDF)
Before this commit: robot 003_cracker_box, 3 links, 2 joints
Links:
- link base_link: mass 0.1 -> 0.411

File: ycb_assets/004_sugar_box/google_16k/004_sugar_box.urdf (robot description, URDF)
Before this commit: robot 004_sugar_box, 3 links, 2 joints
Links:
- link base_link: mass 0.1 -> 0.514

File: ycb_assets/005_tomato_soup_can/google_16k/005_tomato_soup_can.urdf (robot description, URDF)
Before this commit: robot 005_tomato_soup_can, 3 links, 2 joints
Links:
- link base_link: mass 0.1 -> 0.349

File: ycb_assets/006_mustard_bottle/google_16k/006_mustard_bottle.urdf (robot description, URDF)
Before this commit: robot 006_mustard_bottle, 3 links, 2 joints
Links:
- link base_link: mass 0.1 -> 0.603
Joints:
- joint base_to_com: origin xyz=-0.000000 0.000000 0.080734 rpy=0 0 0 -> xyz=0.000000 -0.000000 0.080734 rpy=0 0 0

File: ycb_assets/007_tuna_fish_can/google_16k/007_tuna_fish_can.urdf (robot description, URDF)
Before this commit: robot 007_tuna_fish_can, 3 links, 2 joints
Links:
- link base_link: mass 0.1 -> 0.171

File: ycb_assets/008_pudding_box/google_16k/008_pudding_box.urdf (robot description, URDF)
Before this commit: robot 008_pudding_box, 3 links, 2 joints
Links:
- link base_link: mass 0.1 -> 0.187
Joints:
- joint base_to_com: origin xyz=0.000000 -0.000000 0.018664 rpy=0 0 0 -> xyz=0.000000 0.000000 0.018664 rpy=0 0 0

File: ycb_assets/009_gelatin_box/google_16k/009_gelatin_box.urdf (robot description, URDF)
Before this commit: robot 009_gelatin_box, 3 links, 2 joints
Links:
- link base_link: mass 0.1 -> 0.097
Joints:
- joint base_to_com: origin xyz=0.000000 0.000000 0.013958 rpy=0 0 0 -> xyz=0.000000 -0.000000 0.013958 rpy=0 0 0
- joint base_to_obb: origin xyz=-0.000114 -0.000203 0.014422 rpy=0 0 0 -> xyz=-0.000123 -0.000203 0.014372 rpy=0 0 0

File: ycb_assets/010_potted_meat_can/google_16k/010_potted_meat_can.urdf (robot description, URDF)
Before this commit: robot 010_potted_meat_can, 3 links, 2 joints
Links:
- link base_link: mass 0.1 -> 0.37

File: ycb_assets/011_banana/google_16k/011_banana.urdf (robot description, URDF)
Before this commit: robot 011_banana, 3 links, 2 joints
Links:
- link base_link: mass 0.1 -> 0.066

File: ycb_assets/012_strawberry/google_16k/012_strawberry.urdf (robot description, URDF)
Before this commit: robot 012_strawberry, 3 links, 2 joints
Links:
- link base_link: mass 0.1 -> 0.018
Joints:
- joint base_to_com: origin xyz=-0.000000 0.000000 0.021076 rpy=0 0 0 -> xyz=0.000000 -0.000000 0.021076 rpy=0 0 0

File: ycb_assets/013_apple/google_16k/013_apple.urdf (robot description, URDF)
Before this commit: robot 013_apple, 3 links, 2 joints
Links:
- link base_link: mass 0.1 -> 0.068
Joints:
- joint base_to_com: origin xyz=0.000000 0.000000 0.036490 rpy=0 0 0 -> xyz=-0.000000 -0.000000 0.036490 rpy=0 0 0

File: ycb_assets/014_lemon/google_16k/014_lemon.urdf (robot description, URDF)
Before this commit: robot 014_lemon, 3 links, 2 joints
Links:
- link base_link: mass 0.1 -> 0.029
Joints:
- joint base_to_com: origin xyz=-0.000000 0.000000 0.026204 rpy=0 0 0 -> xyz=0.000000 0.000000 0.026204 rpy=0 0 0

File: ycb_assets/015_peach/google_16k/015_peach.urdf (robot description, URDF)
Before this commit: robot 015_peach, 3 links, 2 joints
Links:
- link base_link: mass 0.1 -> 0.033

File: ycb_assets/016_pear/google_16k/016_pear.urdf (robot description, URDF)
Before this commit: robot 016_pear, 3 links, 2 joints
Links:
- link base_link: mass 0.1 -> 0.049
Joints:
- joint base_to_com: origin xyz=0.000000 -0.000000 0.028412 rpy=0 0 0 -> xyz=0.000000 0.000000 0.028412 rpy=0 0 0

File: ycb_assets/017_orange/google_16k/017_orange.urdf (robot description, URDF)
Before this commit: robot 017_orange, 3 links, 2 joints
Links:
- link base_link: mass 0.1 -> 0.047

File: ycb_assets/018_plum/google_16k/018_plum.urdf (robot description, URDF)
Before this commit: robot 018_plum, 3 links, 2 joints
Links:
- link base_link: mass 0.1 -> 0.025
Joints:
- joint base_to_com: origin xyz=-0.000000 -0.000000 0.023377 rpy=0 0 0 -> xyz=0.000000 -0.000000 0.023377 rpy=0 0 0

File: ycb_assets/019_pitcher_base/google_16k/019_pitcher_base.urdf (robot description, URDF)
Before this commit: robot 019_pitcher_base, 3 links, 2 joints
Links:
- link base_link: mass 0.1 -> 0.178

File: ycb_assets/021_bleach_cleanser/google_16k/021_bleach_cleanser.urdf (robot description, URDF)
Before this commit: robot 021_bleach_cleanser, 3 links, 2 joints
Links:
- link base_link: mass 0.1 -> 1.131

File: ycb_assets/022_windex_bottle/google_16k/022_windex_bottle.urdf (robot description, URDF)
Before this commit: robot 022_windex_bottle, 3 links, 2 joints
Links:
- link base_link: mass 0.1 -> 1.022
Joints:
- joint base_to_com: origin xyz=0.000000 -0.000000 0.111863 rpy=0 0 0 -> xyz=0.000000 0.000000 0.111863 rpy=0 0 0
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